File: Trem_23.kicad_pcb (KiCad board)
At the start: 2 copper layers, 45 x 50 mm, 78 parts, among them J1 +9V, J2 GND, J4 IN GND, J6 OUT GND, J9 IN/LED/GND/OUT, Q1 MMBT5089, Q2 MBT3904DW1, Q3 MBT3904DW1, Q4 MMBT5401, Q5 MMBT3904, SW1 SQ/TRI, SW2 LFO/AUDIO, U1 TL064, U2 CD4053

Commit message: Update Trem_23.kicad_pcb
Parts:
- R26: value 18k -> 20k
- RV4: value 5k -> 2k; footprint Potentiometer_SMD:Potentiometer_Bourns_3314J_Vertical -> Potentiometer_THT:Potentiometer_Bourns_3296W_Vertical
- moved R25 26.8 mm to (62.6, 48.6), turned to 90 degrees
- moved RV4 3.22 mm to (63.2, 42.7), turned to 0 degrees
- moved R10 0.50 mm to (59.9, 46.6)
Connections:
- R24 pad 1: /VA -> Net-(R24-Pad1)
- R25 pad 1: /VA -> Net-(R25-Pad1)
- R26 pad 2: Net-(R26-Pad2) -> /VB
- RV4 pad 1: unconnected-(RV4-Pad1) -> Net-(R24-Pad1)
- RV4 pad 2: /VB -> /VA
- RV4 pad 3: Net-(R26-Pad2) -> Net-(R25-Pad1)
Routing:
- net /VA: track 110.2 -> 0.00 mm, vias 1 -> 0
- net /LED_K: track 72.7 -> 25.6 mm
- net Net-(Q2B-C2): track 37.1 -> 0.00 mm, vias 4 -> 0
- net /VB: track 88.1 -> 65.6 mm
- net /FB: track 32.7 -> 14.8 mm
- net /INT_N: track 40.6 -> 23.4 mm
- net GND: track 216.9 -> 201.9 mm
- net Net-(SW1-A): track 44.3 -> 33.1 mm
- net Net-(R26-Pad2): track 11.1 -> 0.00 mm, vias 2 -> 0
- net /DRV: track 17.4 -> 9.69 mm, vias 2 -> 1
- net /SQR: track 67.9 -> 62.5 mm
- net Net-(Q3A-E1): track 25.8 -> 21.0 mm, vias 2 -> 1
- net /TRI: track 48.2 -> 45.3 mm
Other:
- board text added: "TREM v2.1"
- board text removed: "TREM v2"
