File: Trem_23.kicad_pcb (KiCad board)
At the start: 2 copper layers, 45 x 50 mm, 78 parts, among them J1 +9V, J2 GND, J4 IN GND, J6 OUT GND, J9 IN/LED/GND/OUT, Q1 MMBT5089, Q2 MBT3904DW1, Q3 MBT3904DW1, Q4 MMBT5401, Q5 MMBT3904, SW1 SQ/TRI, SW2 LFO/AUDIO, U1 TL064, U2 CD4053

Commit message: v2.1 PCB: RV4 back to Bourns 3314J (2k SMD, C94513, JLC-placed) for the symmetric balance trim; full re-route; fab files
The 3296W THT trimmer left 24 pads unrouted. 3314J at the v2.0 spot routes cleanly:
0 unconnected, 0 DRC errors, 67 vias.

Co-Authored-By: Claude Opus 5.5 <noreply@anthropic.com>
Parts:
- RV4: footprint Potentiometer_THT:Potentiometer_Bourns_3296W_Vertical -> Potentiometer_SMD:Potentiometer_Bourns_3314J_Vertical
- moved RV4 3.22 mm to (60.0, 42.3), turned to 90 degrees
Routing:
- net /VA: track 0.00 -> 82.5 mm, vias 0 -> 6
- net /LED_K: track 25.6 -> 83.6 mm
- net Net-(R5-Pad1): track 26.8 -> 56.4 mm
- net GND: track 201.9 -> 231.2 mm, vias 1 -> 4
- net Net-(Q2B-C2): track 0.00 -> 28.6 mm, vias 0 -> 4
- net +9V: track 104.8 -> 82.4 mm, vias 2 -> 5
- net /TRI: track 45.3 -> 67.0 mm
- net /FB: track 14.8 -> 36.1 mm
- net Net-(R24-Pad1): track 0.00 -> 20.4 mm, vias 0 -> 2
- net Net-(SW1-A): track 33.1 -> 53.0 mm
- net Net-(U2-C): track 41.0 -> 22.2 mm
- net Net-(D4-A): track 46.3 -> 63.5 mm
- net /SQR: track 62.5 -> 47.9 mm, vias 2 -> 3
- net /LFO: track 34.4 -> 47.7 mm
- net Net-(D3-K): track 41.1 -> 28.2 mm, vias 2 -> 1
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